File: Schematics/FinalLab/reciever.kicad_sch (KiCad schematic)
At the start: 18 parts, among them M1 Stepper_Motor_unipolar_5pin, M2 Motor_DC, SW1 SW_Push, SW2 SW_Push, SW3 SW_Push, U3 NRF24L01, U4 16x2_I2C_LCD, U5 TC74A0-3.3VAT, U6 DHT11, U7 ULN2003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

Commit message: updating
Parts:
- removed D1, D2, D3, D4: LED, symbol Device:LED
- removed U9: LM393, symbol syms:LM293_Optical_Sensor
- added R1: R_Variable_US, symbol Device:R_Variable_US
- added R2: 10k, symbol Device:R_US
- U8: footprint L293D:DIP880W50P254L2000H510Q16 -> Package_DIP:DIP-16_W7.62mm; A_MAX 5.1 -> (none); A_MIN 5.1 -> (none); A_NOM 5.1 -> (none); Availability In Stock -> (none); B_MAX 0.5 -> (none); B_MIN 0.5 -> (none); B_NOM 0.5 -> (none); Check_prices https://www.snapeda.com/parts/L293D/STMicroelectronics/view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 -> (none); D_MAX 20.0 -> (none); D_MIN 20.0 -> (none); D_NOM 20.0 -> (none); Description_1 Bipolar Motor Driver - Parallel 16-PowerDIP -> (none); E1_MAX 7.1 -> (none); E1_MIN 7.1 -> (none); E1_NOM 7.1 -> (none); ENOM 2.54 -> (none); E_NOM 8.8 -> (none); MANUFACTURER ST Microelectronics -> (none); MAXIMUM_PACKAGE_HEIGHT 5.1mm -> (none); MF STMicroelectronics -> (none); MP L293D -> (none); PIN_COUNT 16.0 -> (none); Package DIP-16 STMicroelectronics -> (none); Price None -> (none); STANDARD IPC 7351B -> (none); SnapEDA_Link https://www.snapeda.com/parts/L293D/STMicroelectronics/view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 -> (none)
Connections:
- net LED_DIM_GND is gone; now on net MOSI: A2.26 (D11)
- net +5V: now also U8.16 (VCC1), U8.9 (EN3,4), R2.1; no longer U8.8 (VS)
- net CE: now also A2.22 (D7); no longer A2.23 (D8)
- net CS: now also A2.23 (D8); no longer A2.24 (D9)
- net DHT_DATA: no longer A2.22 (D7)
- net EN1_PWM: now also A2.18 (D3), U8.2 (1A); no longer A2.21 (D6), U8.1 (ENABLE1)
- net GND: now also R1.2
- net IN_1: no longer A2.17 (D2)
- net IN_2: no longer A2.18 (D3)
- net IN_3: no longer A2.19 (D4)
- net IN_4: no longer A2.20 (D5)
- net MISO: now also A2.27 (D12); no longer A2.28 (D13)
- net MOSI: no longer A2.27 (D12)
- net PID_EN: now also A2.21 (D6); no longer A2.12 (A3)
- net SCK: now also A2.28 (D13); no longer A2.25 (D10)
- net V_Batt: now also U8.8 (VCC2); no longer U8.16 (VSS)
- net start: now also A2.19 (D4); no longer A2.9 (A0)
- net stop: now also A2.25 (D10); no longer A2.10 (A1)
- net PIN_X: no longer names the net of A2.15 (D0/RX)
- net PIN_X: no longer U8.2 (INPUT1)
- net PIN_Y: no longer names the net of A2.16 (D1/TX)
- net PIN_Y: no longer U8.7 (INPUT2)
- net en_input: no longer names the net of A2.11 (A2)
- new net EN1_EN2: A2.20 (D5), U8.1 (EN1,2)
- new net EN2_PWM: A2.24 (D9), U8.7 (2A)
- new net ldr_input: A2.9 (A0), R1.1, R2.2
- no-connect marks 13 -> 15
Other:
- note removed: "LED Dimmer"
- moved on the sheet: M2
